Commit message: ros2_hardware_with_gazebo

File: t8_ros_2_controller_hardware/wolf-robot/description/robot.urdf.xacro (robot description, xacro)
@@ -2,4 +2,5 @@
 <robot xmlns:xacro="http://www.ros.org/wiki/xacro"  name="robot">
     <xacro:arg name="use_ros2_control" default="true"/>
+    <xacro:arg name="sim_mode" default="false"/>
     <xacro:include filename="robot_core.xacro"/>
     <xacro:if value="$(arg use_ros2_control)">

File: t8_ros_2_controller_hardware/wolf-robot/description/ros2_control.xacro (robot description, xacro)
@@ -1,90 +1,95 @@
 <?xml version="1.0"?>
 <robot xmlns:xacro="http://www.ros.org/wiki/xacro">
-    <ros2_control name="RealRobot" type="system">
-        <hardware>
-            <plugin>diffdrive_arduino/DiffDriveArduino</plugin>
-            <param name="front_left_wheel_name">front_left_joint</param>
-            <param name="front_right_wheel_name">front_right_joint</param>
-            <param name="back_left_wheel_name">back_left_joint</param>
-            <param name="back_right_wheel_name">back_right_joint</param>
-            <param name="loop_rate">28</param>
-            <param name="device">/dev/ttyUSB0</param>
-            <param name="baud_rate">57600</param>
-            <param name="timeout">1000</param>
-            <param name="enc_counts_per_rev">560</param>
-        </hardware>
-        <joint name="front_left_joint">
-            <command_interface name="velocity">
-                <param name="min">-10</param>
-                <param name="max">10</param>
-            </command_interface>
-            <state_interface name="velocity"/>
-            <state_interface name="position"/>
-        </joint>
-        <joint name="front_right_joint">
-            <command_interface name="velocity">
-                <param name="min">-10</param>
-                <param name="max">10</param>
-            </command_interface>
-            <state_interface name="velocity"/>
-            <state_interface name="position"/>
-        </joint>
-        <joint name="back_left_joint">
-            <command_interface name="velocity">
-                <param name="min">-10</param>
-                <param name="max">10</param>
-            </command_interface>
-            <state_interface name="velocity"/>
-            <state_interface name="position"/>
-        </joint>
-        <joint name="back_right_joint">
-            <command_interface name="velocity">
-                <param name="min">-10</param>
-                <param name="max">10</param>
-            </command_interface>
-            <state_interface name="velocity"/>
-            <state_interface name="position"/>
-        </joint>
-    </ros2_control>
-  <!-- <ros2_control name="GazeboSystem" type="system">
-          <hardware>
-              <plugin>gazebo_ros2_control/GazeboSystem</plugin>
-          </hardware>
-          <joint name="front_left_joint">
-              <command_interface name="velocity">
-                  <param name="min">-10</param>
-                  <param name="max">10</param>
-              </command_interface>
-              <state_interface name="velocity"/>
-              <state_interface name="position"/>
-          </joint>
-          <joint name="front_right_joint">
-              <command_interface name="velocity">
-                  <param name="min">-10</param>
-                  <param name="max">10</param>
-              </command_interface>
-              <state_interface name="velocity"/>
-              <state_interface name="position"/>
-          </joint>
-          <joint name="back_left_joint">
-              <command_interface name="velocity">
-                  <param name="min">-10</param>
-                  <param name="max">10</param>
-              </command_interface>
-              <state_interface name="velocity"/>
-              <state_interface name="position"/>
-          </joint>
-          <joint name="back_right_joint">
-              <command_interface name="velocity">
-                  <param name="min">-10</param>
-                  <param name="max">10</param>
-              </command_interface>
-              <state_interface name="velocity"/>
-              <state_interface name="position"/>
-          </joint>
-      </ros2_control> -->
+    <xacro:unless value="$(arg sim_mode)">
+        <ros2_control name="RealRobot" type="system">
+            <hardware>
+                <plugin>diffdrive_arduino/DiffDriveArduino</plugin>
+                <param name="front_left_wheel_name">front_left_joint</param>
+                <param name="front_right_wheel_name">front_right_joint</param>
+                <param name="back_left_wheel_name">back_left_joint</param>
+                <param name="back_right_wheel_name">back_right_joint</param>
+                <param name="loop_rate">28</param>
+                <param name="device">/dev/ttyUSB0</param>
+                <param name="baud_rate">57600</param>
+                <param name="timeout">1000</param>
+                <param name="enc_counts_per_rev">560</param>
+            </hardware>
+            <joint name="front_left_joint">
+                <command_interface name="velocity">
+                    <param name="min">-10</param>
+                    <param name="max">10</param>
+                </command_interface>
+                <state_interface name="velocity"/>
+                <state_interface name="position"/>
+            </joint>
+            <joint name="front_right_joint">
+                <command_interface name="velocity">
+                    <param name="min">-10</param>
+                    <param name="max">10</param>
+                </command_interface>
+                <state_interface name="velocity"/>
+                <state_interface name="position"/>
+            </joint>
+            <joint name="back_left_joint">
+                <command_interface name="velocity">
+                    <param name="min">-10</param>
+                    <param name="max">10</param>
+                </command_interface>
+                <state_interface name="velocity"/>
+                <state_interface name="position"/>
+            </joint>
+            <joint name="back_right_joint">
+                <command_interface name="velocity">
+                    <param name="min">-10</param>
+                    <param name="max">10</param>
+                </command_interface>
+                <state_interface name="velocity"/>
+                <state_interface name="position"/>
+            </joint>
+        </ros2_control>
+    </xacro:unless>
+    <xacro:if value="$(arg sim_mode)">
+        <ros2_control name="GazeboSystem" type="system">
+                <hardware>
+                    <plugin>gazebo_ros2_control/GazeboSystem</plugin>
+                </hardware>
+                <joint name="front_left_joint">
+                    <command_interface name="velocity">
+                        <param name="min">-10</param>
+                        <param name="max">10</param>
+                    </command_interface>
+                    <state_interface name="velocity"/>
+                    <state_interface name="position"/>
+                </joint>
+                <joint name="front_right_joint">
+                    <command_interface name="velocity">
+                        <param name="min">-10</param>
+                        <param name="max">10</param>
+                    </command_interface>
+                    <state_interface name="velocity"/>
+                    <state_interface name="position"/>
+                </joint>
+                <joint name="back_left_joint">
+                    <command_interface name="velocity">
+                        <param name="min">-10</param>
+                        <param name="max">10</param>
+                    </command_interface>
+                    <state_interface name="velocity"/>
+                    <state_interface name="position"/>
+                </joint>
+                <joint name="back_right_joint">
+                    <command_interface name="velocity">
+                        <param name="min">-10</param>
+                        <param name="max">10</param>
+                    </command_interface>
+                    <state_interface name="velocity"/>
+                    <state_interface name="position"/>
+                </joint>
+            </ros2_control>
+        </xacro:if>
       <gazebo>
           <plugin name="gazebo_ros2_control" filename="libgazebo_ros2_control.so">
               <parameters>$(find wolf-robot)/config/wolf_controller.yaml</parameters>
+              <parameters>$(find wolf-robot)/config/gaz_ros2_ctl_use_sim.yaml</parameters>
           </plugin>
       </gazebo>
